File: Single_LED_channel.kicad_sch (KiCad schematic)
At the start: 5 parts, among them J102 mono-jack, Q103 FQP30N06L

Commit message: V1 for fab
Changed lines of the file:
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@@
   (junction (at 69.215 50.8) (diameter 0) (color 0 0 0 0)
-  )
-  (junction (at 90.17 29.21) (diameter 0) (color 0 0 0 0)
   )
   (junction (at 81.915 50.8) (diameter 0) (color 0 0 0 0)
@@
     (stroke (width 0) (type default))
   )
-  (wire (pts (xy 88.265 31.75) (xy 91.44 31.75))
-    (stroke (width 0) (type default))
-  )
   (wire (pts (xy 106.045 49.53) (xy 106.045 59.055))
     (stroke (width 0) (type default))
@@
     (stroke (width 0) (type default))
   )
-  (wire (pts (xy 106.045 29.21) (xy 106.045 44.45))
+  (wire (pts (xy 106.045 27.94) (xy 106.045 44.45))
     (stroke (width 0) (type default))
   )
@@
     (stroke (width 0) (type default))
   )
-  (wire (pts (xy 90.17 27.305) (xy 90.17 29.21))
-    (stroke (width 0) (type default))
-  )
-  (wire (pts (xy 90.17 29.21) (xy 88.265 29.21))
-    (stroke (width 0) (type default))
-  )
-  (wire (pts (xy 91.44 31.75) (xy 91.44 43.18))
-    (stroke (width 0) (type default))
-  )
-  (wire (pts (xy 90.17 29.21) (xy 106.045 29.21))
+  (wire (pts (xy 91.44 39.37) (xy 91.44 43.18))
     (stroke (width 0) (type default))
   )
@@
     )
   )
-  (symbol (lib_id "power:VDC") (at 90.17 27.305 0) (unit 1)
+  (symbol (lib_id "power:VDC") (at 106.045 27.94 0) (unit 1)
     (in_bom yes) (on_board yes) (dnp no) (fields_autoplaced)
-    (property "Reference" "#PWR0113" (at 90.17 29.845 0)
-      (effects (font (size 1.27 1.27)) hide)
-    )
-    (property "Value" "VDC" (at 90.17 22.225 0)
-      (effects (font (size 1.27 1.27)))
-    )
-    (property "Footprint" "" (at 90.17 27.305 0)
-      (effects (font (size 1.27 1.27)) hide)
-    )
-    (property "Datasheet" "" (at 90.17 27.305 0)
-      (effects (font (size 1.27 1.27)) hide)
-    )
+    (property "Reference" "#PWR0113" (at 106.045 30.48 0)
+      (effects (font (size 1.27 1.27)) hide)
+    )
+    (property "Value" "VDC" (at 106.045 22.86 0)
+      (effects (font (size 1.27 1.27)))
+    )
+    (property "Footprint" "" (at 106.045 27.94 0)
+      (effects (font (size 1.27 1.27)) hide)
+    )
+    (property "Datasheet" "" (at 106.045 27.94 0)
+      (effects (font (size 1.27 1.27)) hide)
+    )
