File: strobe-controller.kicad_sch (KiCad schematic)
At the start: 13 parts, among them J101 Power_in, J102 LED_R, J103 LED_G, J104 LED_W, J105 LED_B, Q105 BSP149

Commit message: V1 for fab
Parts:
- added H103, H104, H105, H106: MountingHole, MountingHole:MountingHole_3.2mm_M3_DIN965, symbol Mechanical:MountingHole
- H101, H102: symbol Mechanical:MountingHole -> Mechanical:DIN_Rail_Adapter
- J102: value LED_R -> LED_B
- J104: value LED_W -> LED_R
- J105: value LED_B -> LED_G
- Q105: jlcpcb (none) -> C534558
Connections:
- net LED_B: now also CO101.Bl; no longer CO101.Gr
- net LED_G: now also CO101.Gr; no longer CO101.Bl
- net VDC: now also D101.1 (+V); no longer D101.5 (+V)
- net drain_B: now also D101.4 (BK), J102.1 (Pin_1); no longer D101.3 (BK), J105.1 (Pin_1)
- net drain_G: now also J105.1 (Pin_1); no longer J103.2 (Pin_2)
- net drain_R: now also D101.3 (RK), J104.2 (Pin_2); no longer D101.1 (RK), J102.1 (Pin_1)
- net drain_W: now also D101.5 (WK), J103.2 (Pin_2); no longer D101.4 (WK), J104.2 (Pin_2)
Other:
- note added: "BSP149H6327XTSA1TR-ND depletion mode NMOS discharge time: RC = 8.8 mF * 500 Ohm = 4.4s discharge curent: 160 mA , 12.8W"
- note added: "Voltage droops during large current pulses Maximum droop allowed: dV/dt = 2 V/ 250 us = 8000 V/s Minimum capacitance per amp: C = I / dV/dt = 0.1 mF Maximum current for large LEDs: 60 A Minimum total capacitance: 6 mF"
- note removed: "BSP149H6327XTSA1TR-ND depletion mode NMOS"
- note removed: "Voltage droops during large current pulses Maximum droop allowed: dV/dt = 100 mV/ 250 us = 400 V/s Minimum capacitance per amp: 2.5 mF Maximum current for 10m of LED strips: 10A Minimum total capacitance: 25mF"
- moved on the sheet: CO101B, CO101C
